Commit message: URDF: regenerate for 11-DOF MVS; fix generator and verifier
generate_urdf.py:
- Ankle pitch joint inserted between shin and foot per leg
- Hip roll and hip pitch now separate revolute joints (previously
  hip roll was silently dropped)
- All joint axis directions read from kinematics.yaml, not hardcoded
- All joint limits read from joints.yaml, not hardcoded
- Hip lateral offset read from geometry.yaml twin-rail spacing
- Torso now three proper revolute joints (pitch, roll, yaw)
- Ankle inclusion driven by is_mvs_actuated() check — URDF follows
  YAML automatically if scope changes again
- Fixed foot joint origin to use full ankle_to_sole_offset, not half

verify_urdf_dimensions.py:
- Updated joint name lookups to match new naming convention
  (knee_pitch_joint, ankle_pitch_joint, foot_joint)
- Measurement logic now correctly walks three-segment chain:
  thigh / shin / ankle-to-sole

File: simulation/urdf/megadroid_mvs.urdf (robot description, URDF)
Before this commit: robot megadroid_mvs, 12 links, 11 joints
Links:
- removed link left_hip
- removed link left_knee
- removed link right_hip
- removed link right_knee
- added link left_ankle; visual sphere radius=0.025
- added link left_hip_roll_link; visual sphere radius=0.03
- added link right_ankle; visual sphere radius=0.025
- added link right_hip_roll_link; visual sphere radius=0.03
- added link torso_pitch_link; visual box size=0.05 0.20 0.05
- added link torso_roll_link; visual box size=0.05 0.20 0.05
- link left_thigh: geometry visual cylinder length=0.3 radius=0.040
- link pelvis: geometry visual box size=0.20 0.30 0.15
- link right_thigh: geometry visual cylinder length=0.3 radius=0.040
- link torso: geometry visual box size=0.15 0.25 0.40
Joints:
- removed joint left_hip_joint
- removed joint left_knee_joint
- removed joint left_shin_joint
- removed joint left_thigh_joint
- removed joint pelvis_to_torso
- removed joint right_hip_joint
- removed joint right_knee_joint
- removed joint right_shin_joint
- removed joint right_thigh_joint
- added joint left_ankle_pitch_joint: type revolute, parent left_shin, child left_ankle, origin xyz=0 0 -0.3 rpy=0 0 0, axis 0 1 0, limit lower=-0.5235987755982988 upper=0.5235987755982988 effort=100.0 velocity=1.0
- added joint left_hip_pitch_joint: type revolute, parent left_hip_roll_link, child left_thigh, origin xyz=0 0 0 rpy=0 0 0, axis 0 1 0, limit lower=-0.5235987755982988 upper=1.9198621771937625 effort=100.0 velocity=1.0
- added joint left_hip_roll_joint: type revolute, parent pelvis, child left_hip_roll_link, origin xyz=0 0.05 0 rpy=0 0 0, axis 1 0 0, limit lower=-0.5235987755982988 upper=0.5235987755982988 effort=100.0 velocity=1.0
- added joint left_knee_pitch_joint: type revolute, parent left_thigh, child left_shin, origin xyz=0 0 -0.3 rpy=0 0 0, axis 0 1 0, limit lower=0.0 upper=2.443460952792061 effort=100.0 velocity=1.0
- added joint right_ankle_pitch_joint: type revolute, parent right_shin, child right_ankle, origin xyz=0 0 -0.3 rpy=0 0 0, axis 0 1 0, limit lower=-0.5235987755982988 upper=0.5235987755982988 effort=100.0 velocity=1.0
- added joint right_hip_pitch_joint: type revolute, parent right_hip_roll_link, child right_thigh, origin xyz=0 0 0 rpy=0 0 0, axis 0 1 0, limit lower=-0.5235987755982988 upper=1.9198621771937625 effort=100.0 velocity=1.0
- added joint right_hip_roll_joint: type revolute, parent pelvis, child right_hip_roll_link, origin xyz=0 -0.05 0 rpy=0 0 0, axis 1 0 0, limit lower=-0.5235987755982988 upper=0.5235987755982988 effort=100.0 velocity=1.0
- added joint right_knee_pitch_joint: type revolute, parent right_thigh, child right_shin, origin xyz=0 0 -0.3 rpy=0 0 0, axis 0 1 0, limit lower=0.0 upper=2.443460952792061 effort=100.0 velocity=1.0
- added joint torso_pitch_joint: type revolute, parent pelvis, child torso_pitch_link, origin xyz=0 0 0.075 rpy=0 0 0, axis 0 1 0, limit lower=-0.5235987755982988 upper=0.5235987755982988 effort=100.0 velocity=1.0
- added joint torso_roll_joint: type revolute, parent torso_pitch_link, child torso_roll_link, origin xyz=0 0 0 rpy=0 0 0, axis 1 0 0, limit lower=-0.3490658503988659 upper=0.3490658503988659 effort=100.0 velocity=1.0
- added joint torso_yaw_joint: type revolute, parent torso_roll_link, child torso, origin xyz=0 0 0 rpy=0 0 0, axis 0 0 1, limit lower=-0.7853981633974483 upper=0.7853981633974483 effort=100.0 velocity=1.0
- joint left_foot_joint: origin xyz=0 0 -0.38 rpy=0 0 0 -> xyz=0.05 0 -0.08 rpy=0 0 0; parent left_shin -> left_ankle
- joint right_foot_joint: origin xyz=0 0 -0.38 rpy=0 0 0 -> xyz=0.05 0 -0.08 rpy=0 0 0; parent right_shin -> right_ankle
