Commit message: P3: add MuJoCo simulation foundation (mass, MJCF generator, load test)
design/mass.yaml (new):
  Authoritative mass estimates per link — 8.9 kg total. Nominal values
  based on 775 DC motor assemblies + structural framing; to be verified
  during P6 physical build.

tools/generate_urdf.py (updated):
  Now reads mass.yaml and emits <inertial> elements for every link.
  Adds box_inertia/cylinder_inertia/sphere_inertia helpers. URDF is now
  dynamics-capable and loads cleanly in MuJoCo. Signature updated:
  create_urdf(..., mass_data).

tools/generate_mjcf.py (new):
  Generates simulation/mujoco/megadroid_mvs.xml from all four design
  YAML files. Produces a complete MuJoCo scene: floating pelvis with
  freejoint, explicit inertial elements, position actuators for all 11
  MVS joints (kp=150), foot contact geometry, ground plane, and sensors
  for pelvis/foot positions. Verified: 15 bodies, 17 DOF, 11 actuators,
  8.90 kg total mass.

tools/sim_load_test.py (new):
  Quick sanity check — loads MJCF, prints model statistics, runs one
  physics step. Passes cleanly.

simulation/urdf/megadroid_mvs.urdf (regenerated):
  Now includes <inertial> elements; dynamics-capable.

simulation/mujoco/megadroid_mvs.xml (generated):
  MuJoCo scene file; do not edit — regenerate with generate_mjcf.py.

P3 standing validation (sim_standing.py) is in progress — freejoint
initialization needs a fix before the standing test is meaningful.

Co-Authored-By: Claude Sonnet 4.6 <noreply@anthropic.com>

File: simulation/urdf/megadroid_mvs.urdf (robot description, URDF)
Before this commit: robot megadroid_mvs, 14 links, 13 joints
Links:
- link left_ankle: mass None -> 0.35
- link left_foot: mass None -> 0.15
- link left_hip_roll_link: mass None -> 0.3
- link left_shin: mass None -> 0.7
- link left_thigh: mass None -> 0.9
- link pelvis: mass None -> 1.5
- link right_ankle: mass None -> 0.35
- link right_foot: mass None -> 0.15
- link right_hip_roll_link: mass None -> 0.3
- link right_shin: mass None -> 0.7
- link right_thigh: mass None -> 0.9
- link torso: mass None -> 2.0
- link torso_pitch_link: mass None -> 0.3
- link torso_roll_link: mass None -> 0.3

Commit message: Docs: rehydrate SPEC/MECH/README, regenerate URDF/MJCF for ankle_roll
Mechanical output of the previous two commits: SPEC.md now correctly
shows 11 actuated DOF (was 9) with Ankle Pitch listed, describes the
flat sole plate and passive ankle_roll instead of the never-actually-
simulated "ball foot". MECH.md's structural stack, DOF count, and F/T
sensor section updated to match. URDF and MJCF regenerated — 17 bodies
(was 15), still 11 actuators, dimensions still match design/geometry.yaml
exactly.

Co-Authored-By: Claude Sonnet 5 <noreply@anthropic.com>
Claude-Session: https://claude.ai/code/session_01AHR3z3mgUGSG2NVo8EEy6h

File: simulation/urdf/megadroid_mvs.urdf (robot description, URDF)
Before this commit: robot megadroid_mvs, 14 links, 13 joints
Links:
- added link left_ankle_roll, mass 0.05; visual sphere radius=0.020
- added link right_ankle_roll, mass 0.05; visual sphere radius=0.020
Joints:
- added joint left_ankle_roll_joint: type revolute, parent left_ankle, child left_ankle_roll, origin xyz=0 0 0 rpy=0 0 0, axis 1 0 0, limit lower=-0.2617993877991494 upper=0.2617993877991494 effort=100.0 velocity=1.0
- added joint right_ankle_roll_joint: type revolute, parent right_ankle, child right_ankle_roll, origin xyz=0 0 0 rpy=0 0 0, axis 1 0 0, limit lower=-0.2617993877991494 upper=0.2617993877991494 effort=100.0 velocity=1.0
- joint left_foot_joint: parent left_ankle -> left_ankle_roll
- joint right_foot_joint: parent right_ankle -> right_ankle_roll

Commit message: URDF/MJCF: regenerate for ankle_roll actuation
ankle_roll drops its <joint stiffness>/<joint springref> attributes
(no longer passive) and gains a position actuator, generated
automatically by the existing actuated+MVS filter in generate_mjcf.py
-- no generator code changes were needed. Verified via
verify_urdf_dimensions.py (leg lengths unchanged, ankle_roll's z-offset
still zero) and sim_load_test.py (17 bodies, 13 actuators, 9.60kg).

Co-Authored-By: Claude Sonnet 5 <noreply@anthropic.com>
Claude-Session: https://claude.ai/code/session_01AHR3z3mgUGSG2NVo8EEy6h

File: simulation/urdf/megadroid_mvs.urdf (robot description, URDF)
Before this commit: robot megadroid_mvs, 16 links, 15 joints
Links:
- link left_ankle_roll: mass 0.05 -> 0.35
- link right_ankle_roll: mass 0.05 -> 0.35

Commit message: Models: regenerate URDF and MJCF with joint torque limits and the pelvis IMU
MJCF: forcerange +/-2.8 N-m on all 13 position actuators (previously
absent -- unbounded torque), plus imu_site at the pelvis body origin with
gyro and accelerometer sensors.

URDF: joint limits now carry the real effort (2.8 N-m) and velocity
(78.5 rad/s) from design/actuation.yaml, replacing the placeholder
effort=100.0 / velocity=1.0.

Verified: verify_urdf_dimensions.py passes, sim_load_test.py loads and
steps the model with all 13 actuators.

Co-Authored-By: Claude Opus 5 <noreply@anthropic.com>
Claude-Session: https://claude.ai/code/session_01JfjyLTEHtH1Vw7kgW9Vbj4

File: simulation/urdf/megadroid_mvs.urdf (robot description, URDF)
Before this commit: robot megadroid_mvs, 16 links, 15 joints
Joints:
- joint left_ankle_pitch_joint: limit lower=-0.5235987755982988 upper=0.5235987755982988 effort=100.0 velocity=1.0 -> lower=-0.5235987755982988 upper=0.5235987755982988 effort=2.8 velocity=78.5
- joint left_ankle_roll_joint: limit lower=-0.2617993877991494 upper=0.2617993877991494 effort=100.0 velocity=1.0 -> lower=-0.2617993877991494 upper=0.2617993877991494 effort=2.8 velocity=78.5
- joint left_hip_pitch_joint: limit lower=-0.5235987755982988 upper=1.9198621771937625 effort=100.0 velocity=1.0 -> lower=-0.5235987755982988 upper=1.9198621771937625 effort=2.8 velocity=78.5
- joint left_hip_roll_joint: limit lower=-0.5235987755982988 upper=0.5235987755982988 effort=100.0 velocity=1.0 -> lower=-0.5235987755982988 upper=0.5235987755982988 effort=2.8 velocity=78.5
- joint left_knee_pitch_joint: limit lower=0.0 upper=2.443460952792061 effort=100.0 velocity=1.0 -> lower=0.0 upper=2.443460952792061 effort=2.8 velocity=78.5
- joint right_ankle_pitch_joint: limit lower=-0.5235987755982988 upper=0.5235987755982988 effort=100.0 velocity=1.0 -> lower=-0.5235987755982988 upper=0.5235987755982988 effort=2.8 velocity=78.5
- joint right_ankle_roll_joint: limit lower=-0.2617993877991494 upper=0.2617993877991494 effort=100.0 velocity=1.0 -> lower=-0.2617993877991494 upper=0.2617993877991494 effort=2.8 velocity=78.5
- joint right_hip_pitch_joint: limit lower=-0.5235987755982988 upper=1.9198621771937625 effort=100.0 velocity=1.0 -> lower=-0.5235987755982988 upper=1.9198621771937625 effort=2.8 velocity=78.5
- joint right_hip_roll_joint: limit lower=-0.5235987755982988 upper=0.5235987755982988 effort=100.0 velocity=1.0 -> lower=-0.5235987755982988 upper=0.5235987755982988 effort=2.8 velocity=78.5
- joint right_knee_pitch_joint: limit lower=0.0 upper=2.443460952792061 effort=100.0 velocity=1.0 -> lower=0.0 upper=2.443460952792061 effort=2.8 velocity=78.5
- joint torso_pitch_joint: limit lower=-0.5235987755982988 upper=0.5235987755982988 effort=100.0 velocity=1.0 -> lower=-0.5235987755982988 upper=0.5235987755982988 effort=2.8 velocity=78.5
- joint torso_roll_joint: limit lower=-0.3490658503988659 upper=0.3490658503988659 effort=100.0 velocity=1.0 -> lower=-0.3490658503988659 upper=0.3490658503988659 effort=2.8 velocity=78.5
- joint torso_yaw_joint: limit lower=-0.7853981633974483 upper=0.7853981633974483 effort=100.0 velocity=1.0 -> lower=-0.7853981633974483 upper=0.7853981633974483 effort=2.8 velocity=78.5

Commit message: Models: regenerate URDF and MJCF at the 80:1 envelope
forcerange +-11.2 N-m on all 13 actuators (was +-2.8); URDF joint limits
effort 11.2 N-m, velocity 19.6 rad/s. Verified: verify_urdf_dimensions
passes, sim_load_test loads and steps.

Co-Authored-By: Claude Opus 5 <noreply@anthropic.com>
Claude-Session: https://claude.ai/code/session_01JfjyLTEHtH1Vw7kgW9Vbj4

File: simulation/urdf/megadroid_mvs.urdf (robot description, URDF)
Before this commit: robot megadroid_mvs, 16 links, 15 joints
Joints:
- joint left_ankle_pitch_joint: limit lower=-0.5235987755982988 upper=0.5235987755982988 effort=2.8 velocity=78.5 -> lower=-0.5235987755982988 upper=0.5235987755982988 effort=11.2 velocity=19.6
- joint left_ankle_roll_joint: limit lower=-0.2617993877991494 upper=0.2617993877991494 effort=2.8 velocity=78.5 -> lower=-0.2617993877991494 upper=0.2617993877991494 effort=11.2 velocity=19.6
- joint left_hip_pitch_joint: limit lower=-0.5235987755982988 upper=1.9198621771937625 effort=2.8 velocity=78.5 -> lower=-0.5235987755982988 upper=1.9198621771937625 effort=11.2 velocity=19.6
- joint left_hip_roll_joint: limit lower=-0.5235987755982988 upper=0.5235987755982988 effort=2.8 velocity=78.5 -> lower=-0.5235987755982988 upper=0.5235987755982988 effort=11.2 velocity=19.6
- joint left_knee_pitch_joint: limit lower=0.0 upper=2.443460952792061 effort=2.8 velocity=78.5 -> lower=0.0 upper=2.443460952792061 effort=11.2 velocity=19.6
- joint right_ankle_pitch_joint: limit lower=-0.5235987755982988 upper=0.5235987755982988 effort=2.8 velocity=78.5 -> lower=-0.5235987755982988 upper=0.5235987755982988 effort=11.2 velocity=19.6
- joint right_ankle_roll_joint: limit lower=-0.2617993877991494 upper=0.2617993877991494 effort=2.8 velocity=78.5 -> lower=-0.2617993877991494 upper=0.2617993877991494 effort=11.2 velocity=19.6
- joint right_hip_pitch_joint: limit lower=-0.5235987755982988 upper=1.9198621771937625 effort=2.8 velocity=78.5 -> lower=-0.5235987755982988 upper=1.9198621771937625 effort=11.2 velocity=19.6
- joint right_hip_roll_joint: limit lower=-0.5235987755982988 upper=0.5235987755982988 effort=2.8 velocity=78.5 -> lower=-0.5235987755982988 upper=0.5235987755982988 effort=11.2 velocity=19.6
- joint right_knee_pitch_joint: limit lower=0.0 upper=2.443460952792061 effort=2.8 velocity=78.5 -> lower=0.0 upper=2.443460952792061 effort=11.2 velocity=19.6
- joint torso_pitch_joint: limit lower=-0.5235987755982988 upper=0.5235987755982988 effort=2.8 velocity=78.5 -> lower=-0.5235987755982988 upper=0.5235987755982988 effort=11.2 velocity=19.6
- joint torso_roll_joint: limit lower=-0.3490658503988659 upper=0.3490658503988659 effort=2.8 velocity=78.5 -> lower=-0.3490658503988659 upper=0.3490658503988659 effort=11.2 velocity=19.6
- joint torso_yaw_joint: limit lower=-0.7853981633974483 upper=0.7853981633974483 effort=2.8 velocity=78.5 -> lower=-0.7853981633974483 upper=0.7853981633974483 effort=11.2 velocity=19.6

Commit message: URDF/MJCF: regenerate for 175 mm hip spacing
Co-Authored-By: Claude Sonnet 5.5 <noreply@anthropic.com>
Claude-Session: https://claude.ai/code/session_01JfjyLTEHtH1Vw7kgW9Vbj4

File: simulation/urdf/megadroid_mvs.urdf (robot description, URDF)
Before this commit: robot megadroid_mvs, 16 links, 15 joints
Joints:
- joint left_hip_roll_joint: origin xyz=0 0.05 0 rpy=0 0 0 -> xyz=0 0.0875 0 rpy=0 0 0
- joint right_hip_roll_joint: origin xyz=0 -0.05 0 rpy=0 0 0 -> xyz=0 -0.0875 0 rpy=0 0 0

Commit message: Simulation: regenerate URDF and MJCF with hip yaw joints
Co-Authored-By: Claude Sonnet 5.5 <noreply@anthropic.com>
Claude-Session: https://claude.ai/code/session_01JfjyLTEHtH1Vw7kgW9Vbj4

File: simulation/urdf/megadroid_mvs.urdf (robot description, URDF)
Before this commit: robot megadroid_mvs, 16 links, 15 joints
Links:
- added link left_hip_yaw_link, mass 0.5; visual sphere radius=0.03
- added link right_hip_yaw_link, mass 0.5; visual sphere radius=0.03
Joints:
- added joint left_hip_yaw_joint: type revolute, parent pelvis, child left_hip_yaw_link, origin xyz=0 0.0875 0 rpy=0 0 0, axis 0 0 1, limit lower=-0.5235987755982988 upper=0.5235987755982988 effort=11.2 velocity=19.6
- added joint right_hip_yaw_joint: type revolute, parent pelvis, child right_hip_yaw_link, origin xyz=0 -0.0875 0 rpy=0 0 0, axis 0 0 1, limit lower=-0.5235987755982988 upper=0.5235987755982988 effort=11.2 velocity=19.6
- joint left_hip_roll_joint: origin xyz=0 0.0875 0 rpy=0 0 0 -> xyz=0 0 0 rpy=0 0 0; parent pelvis -> left_hip_yaw_link
- joint right_hip_roll_joint: origin xyz=0 -0.0875 0 rpy=0 0 0 -> xyz=0 0 0 rpy=0 0 0; parent pelvis -> right_hip_yaw_link
